File: ETH_Port.kicad_sch (KiCad schematic)
At the start: 4 parts

Commit message: .
Parts:
- RJ1: footprint da:RJ45-TH_HR911130A -> easyeda2kicad:RJ45-TH_HR911130A
Changed lines of the file:
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@@
 			)
 		)
-		(property "Footprint" "da:RJ45-TH_HR911130A"
+		(property "Footprint" "easyeda2kicad:RJ45-TH_HR911130A"
 			(at 160.02 137.16 0)
 			(effects
