File: Power Lines.kicad_sch (KiCad schematic)
At the start: 25 parts, among them U4 TLV70233DBVR

Commit message: .
Parts:
- U4: footprint da:SOT-23-5_L3.0-W1.7-P0.95-LS2.8-BR -> easyeda2kicad:SOT-23-5_L3.0-W1.7-P0.95-LS2.8-BR
Changed lines of the file:
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@@
 			)
 		)
-		(property "Footprint" "da:SOT-23-5_L3.0-W1.7-P0.95-LS2.8-BR"
+		(property "Footprint" "easyeda2kicad:SOT-23-5_L3.0-W1.7-P0.95-LS2.8-BR"
 			(at 241.3 71.12 0)
 			(effects
