File: USB 3.2 gen 1 to Gigabit Ethernet.kicad_pcb (KiCad board)
At the start: 4 copper layers, 50 x 27.5 mm, 54 parts, among them U1 VL162, U2 RTL8153-VC-CG, U3 W25Q16BVSSIG, U4 TLV70233DBVR, Y1 25Mhz

Commit message: .
Parts:
- RJ1: footprint da:RJ45-TH_HR911130A -> easyeda2kicad:RJ45-TH_HR911130A
- U1: footprint da:MQFN-28_L4.5-W3.5-P0.40-BL-EP -> easyeda2kicad:MQFN-28_L4.5-W3.5-P0.40-BL-EP
- U2: footprint da:QFN-48_L6.0-W6.0-P0.40-TL-EP4.4 -> easyeda2kicad:QFN-48_L6.0-W6.0-P0.40-TL-EP4.4
- U3: footprint da:SOIC-8_L5.3-W5.3-P1.27-LS8.0-BL -> easyeda2kicad:SOIC-8_L5.3-W5.3-P1.27-LS8.0-BL
- U4: footprint da:SOT-23-5_L3.0-W1.7-P0.95-LS2.8-BR -> easyeda2kicad:SOT-23-5_L3.0-W1.7-P0.95-LS2.8-BR
- USB1: footprint da:USB-C-SMD_TYPEC-324-BCP24 -> easyeda2kicad:USB-C-SMD_TYPEC-324-BCP24
Routing:
- net D-: track 39.2 -> 40.7 mm
