File: USB 3.2 gen 1 to Gigabit Ethernet.kicad_sch (KiCad schematic)
At the start: 11 parts, among them U2 RTL8153-VC-CG, U3 W25Q16BVSSIG, Y1 25Mhz

Commit message: .
Parts:
- U2: footprint da:QFN-48_L6.0-W6.0-P0.40-TL-EP4.4 -> easyeda2kicad:QFN-48_L6.0-W6.0-P0.40-TL-EP4.4
- U3: footprint da:SOIC-8_L5.3-W5.3-P1.27-LS8.0-BL -> easyeda2kicad:SOIC-8_L5.3-W5.3-P1.27-LS8.0-BL
Changed lines of the file:
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@@
 			)
 		)
-		(property "Footprint" "da:QFN-48_L6.0-W6.0-P0.40-TL-EP4.4"
+		(property "Footprint" "easyeda2kicad:QFN-48_L6.0-W6.0-P0.40-TL-EP4.4"
 			(at 194.31 138.43 0)
 			(effects
@@
 			)
 		)
-		(property "Footprint" "da:SOIC-8_L5.3-W5.3-P1.27-LS8.0-BL"
+		(property "Footprint" "easyeda2kicad:SOIC-8_L5.3-W5.3-P1.27-LS8.0-BL"
 			(at 59.69 138.43 0)
 			(effects
