File: USB Circuit .kicad_sch (KiCad schematic)
At the start: 13 parts, among them U1 VL162

Commit message: .
Parts:
- U1: footprint da:MQFN-28_L4.5-W3.5-P0.40-BL-EP -> easyeda2kicad:MQFN-28_L4.5-W3.5-P0.40-BL-EP
- USB1: footprint da:USB-C-SMD_TYPEC-324-BCP24 -> easyeda2kicad:USB-C-SMD_TYPEC-324-BCP24
Changed lines of the file:
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@@
 			)
 		)
-		(property "Footprint" "da:USB-C-SMD_TYPEC-324-BCP24"
+		(property "Footprint" "easyeda2kicad:USB-C-SMD_TYPEC-324-BCP24"
 			(at 160.02 160.02 0)
 			(effects
@@
 			)
 		)
-		(property "Footprint" "da:MQFN-28_L4.5-W3.5-P0.40-BL-EP"
+		(property "Footprint" "easyeda2kicad:MQFN-28_L4.5-W3.5-P0.40-BL-EP"
 			(at 173.99 88.9 0)
 			(effects
